File: Hardware/ORBIT.kicad_sch (KiCad schematic)
At the start: 52 parts, among them J1 West Connector, J2 East Connector, U1 MCP73031, U10 8MHz, U15 TPS63802DLAR, U16 STM32F030C8Tx, U22 CP2102-GMR

Commit message: Version 1.0
Parts:
- BOOT0: renamed from BOOT1; LCSC Part # C145858 -> C145857
- PWR1: value PWR_SW -> PWR; LCSC Part # C145858 -> C145857
- SW1: renamed from RESET1; value SW_Push -> RESET
- SW2: renamed from USER1; value SW_Push -> USER
Changed lines of the file:
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@@
   (symbol (lib_id "Korean Hroparts Elec SPDT:K3-1270L-F1") (at 49.53 49.53 0) (mirror y) (unit 1)
     (in_bom yes) (on_board yes) (dnp no)
-    (property "Reference" "BOOT1" (at 49.53 54.61 0)
+    (property "Reference" "BOOT0" (at 49.53 54.61 0)
       (effects (font (size 1.27 1.27)))
     )
@@
       (effects (font (size 1.27 1.27)) hide)
     )
-    (property "LCSC Part #" "C145858" (at 49.53 49.53 0)
+    (property "LCSC Part #" "C145857" (at 49.53 49.53 0)
       (effects (font (size 1.27 1.27)) hide)
     )
@@
       (project "ORBIT"
         (path "/3070b2ed-24f5-4699-8606-a941013223e7"
-          (reference "BOOT1") (unit 1)
+          (reference "BOOT0") (unit 1)
         )
       )
@@
   (symbol (lib_id "Switch:SW_Push") (at 85.09 40.64 90) (unit 1)
     (in_bom yes) (on_board yes) (dnp no) (fields_autoplaced)
-    (property "Reference" "RESET1" (at 86.36 39.37 90)
+    (property "Reference" "SW1" (at 86.36 39.37 90)
       (effects (font (size 1.27 1.27)) (justify right))
     )
-    (property "Value" "SW_Push" (at 86.36 41.91 90)
+    (property "Value" "RESET" (at 86.36 41.91 90)
       (effects (font (size 1.27 1.27)) (justify right))
     )
@@
       (project "ORBIT"
         (path "/3070b2ed-24f5-4699-8606-a941013223e7"
-          (reference "RESET1") (unit 1)
+          (reference "SW1") (unit 1)
         )
       )
@@
   (symbol (lib_id "Switch:SW_Push") (at 33.02 116.84 0) (unit 1)
     (in_bom yes) (on_board yes) (dnp no) (fields_autoplaced)
-    (property "Reference" "USER1" (at 33.02 108.458 0)
-      (effects (font (size 1.27 1.27)))
-    )
-    (property "Value" "SW_Push" (at 33.02 110.998 0)
+    (property "Reference" "SW2" (at 33.02 109.22 0)
+      (effects (font (size 1.27 1.27)))
+    )
+    (property "Value" "USER" (at 33.02 111.76 0)
       (effects (font (size 1.27 1.27)))
     )
@@
       (project "ORBIT"
         (path "/3070b2ed-24f5-4699-8606-a941013223e7"
-          (reference "USER1") (unit 1)
+          (reference "SW2") (unit 1)
         )
       )
@@
       (effects (font (size 1.27 1.27)) (justify right))
     )
-    (property "Value" "PWR_SW" (at 266.7 22.606 90)
+    (property "Value" "PWR" (at 266.7 22.606 90)
       (effects (font (size 1.27 1.27)))
     )
@@
       (effects (font (size 1.27 1.27)) hide)
     )
-    (property "LCSC Part #" "C145858" (at 257.81 22.606 90)
-      (effects (font (size 1.27 1.27)) hide)
-    )
+    (property "LCSC Part #" "C145857" (at 257.81 22.606 90)
+      (effects (font (size 1.27 1.27)) hide)
+    )
